Commit message: change camera position

File: turtlebot_description/urdf/turtlebot_properties.urdf.xacro (robot description, xacro)
@@ -19,7 +19,8 @@
      (currently in development and awaiting feedback)
    -->
-	<xacro:property name="cam_px" value="-0.087" />
-<!--	<xacro:property name="cam_py" value="-0.0125" /> Y varies for different configurations. get sets in sensors_urdf -->
-	<xacro:property name="cam_pz" value="0.2870" />
+	<xacro:property name="cam_px" value="0.2000" />
+<!--	<xacro:property name="cam_py" value="-0.0125" /> Y varies for different
+configurations. get sets in sensors_urdf -->
+	<xacro:property name="cam_pz" value="0.3000" />
 	<xacro:property name="cam_or" value="0" />
 	<xacro:property name="cam_op" value="0" />
